Commit message: Wrote gazebo_control and driven the libot in gazebo

File: description/gazebo_control.xacro (robot description, xacro)
@@ -2,19 +2,27 @@
 <robot xmlns:xacro="http://www.ros.org/wiki/xacro">
     <gazebo>
-        <plugin name="diff_drive" filename="libgazebo_ros_diff_drive.so">
-            <!-- Wheel Information -->
-            <left_joint>left_wheel_joint</left_joint>
-            <right_joint>right_wheel_joint</right_joint>
-            <wheel_separation>0.297</wheel_separation>
-            <wheel_diameter>0.066</wheel_diameter>
-            <!-- Limits -->
-            <max_wheel_torque>200</max_wheel_torque>
-            <max_wheel_acceleration>10.0</max_wheel_acceleration>
-            <!-- Output -->
-            <odometry_frame>odom</odometry_frame>
-            <robot_base_frame>base_link</robot_base_frame>
-            <publish_odom>true</publish_odom>
-            <publish_odom_tf>true</publish_odom_tf>
-            <publish_wheel_tf>true</publish_wheel_tf>
+        <plugin name='skid_steer_drive' filename='libgazebo_ros_diff_drive.so'>
+        <!-- Number of wheel pairs -->
+        <num_wheel_pairs>2</num_wheel_pairs>
+        <!-- wheels0 -->
+        <left_joint>front_left_wheel_joint</left_joint>
+        <right_joint>front_right_wheel_joint</right_joint>
+        <!-- wheels1-->
+        <left_joint>rear_left_wheel_joint</left_joint>
+        <right_joint>rear_right_wheel_joint</right_joint>
+        <!-- kinematics -->
+        <wheel_separation>0.14</wheel_separation>
+        <wheel_separation>0.14</wheel_separation>
+        <wheel_diameter>0.05</wheel_diameter>
+        <wheel_diameter>0.05</wheel_diameter>
+        <!-- limits -->
+        <max_wheel_torque>20</max_wheel_torque>
+        <max_wheel_acceleration>1.0</max_wheel_acceleration>
+        <!-- output -->
+        <publish_odom>true</publish_odom>
+        <publish_odom_tf>true</publish_odom_tf>
+        <publish_wheel_tf>true</publish_wheel_tf>
+        <odometry_frame>odom</odometry_frame>
+        <robot_base_frame>base_link</robot_base_frame>
         </plugin>
     </gazebo>

File: description/robot.urdf.xacro (robot description, xacro)
@@ -1,13 +1,5 @@
 <?xml version="1.0"?>
 <robot xmlns:xacro="http://www.ros.org/wiki/xacro"  name="robot">
-    <xacro:arg name="use_ros2_control" default="true"/>
-    <xacro:arg name="sim_mode" default="false"/>
     <xacro:include filename="robot_core.xacro" />
-    <xacro:if value="$(arg use_ros2_control)">
-        <xacro:include filename="ros2_control.xacro" />
-    </xacro:if>
-    <xacro:unless value="$(arg use_ros2_control)">
-        <xacro:include filename="gazebo_control.xacro" />
-    </xacro:unless>
-    <xacro:include filename="lidar.xacro" />
+    <xacro:include filename="gazebo_control.xacro" />
 </robot>

File: description/robot_core.xacro (robot description, xacro)
@@ -2,14 +2,13 @@
 <robot xmlns:xacro="http://www.ros.org/wiki/xacro" >
     <xacro:include filename="inertial_macros.xacro"/>
-    <xacro:property name="chassis_length" value="0.22"/>
+    <xacro:property name="chassis_length" value="0.24"/>
     <xacro:property name="chassis_width" value="0.12"/>
-    <xacro:property name="chassis_height" value="0.12"/>
-    <xacro:property name="chassis_mass" value="0.5"/>
+    <xacro:property name="chassis_height" value="0.10"/>
+    <xacro:property name="chassis_mass" value="0.800"/>
     <xacro:property name="wheel_radius" value="0.025"/>
     <xacro:property name="wheel_thickness" value="0.020"/>
-    <xacro:property name="wheel_mass" value="0.04"/>
-    <xacro:property name="wheel_offset_x" value="0.040"/>
+    <xacro:property name="wheel_mass" value="0.050"/>
+    <xacro:property name="wheel_offset_x" value="0.075"/>
     <xacro:property name="wheel_offset_y" value="0.070"/>
-    <xacro:property name="wheel_offset_z" value="0.025"/>
     <material name="white">
         <color rgba="1 1 1 1" />
@@ -30,17 +29,9 @@
     <link name="base_link">
     </link>
-    <!-- BASE_FOOTPRINT LINK -->
-    <joint name="base_footprint_joint" type="fixed">
-        <parent link="base_link"/>
-        <child link="base_footprint"/>
-        <origin xyz="0 0 0" rpy="0 0 0"/>
-    </joint>
-    <link name="base_footprint">
-    </link>
     <!-- CHASSIS LINK -->
     <joint name="chassis_joint" type="fixed">
         <parent link="base_link"/>
         <child link="chassis"/>
-        <origin xyz="0 0 ${chassis_height/2 + wheel_offset_z}"/>
+        <origin xyz="0 0 0"/>
     </joint>
     <link name="chassis">
@@ -58,10 +49,10 @@
             </geometry>
         </collision>
-        <xacro:inertial_box mass="0.5" x="${chassis_length}" y="${chassis_width}" z="${chassis_height}">
-            <origin xyz="${chassis_length/2} 0 ${chassis_height/2}" rpy="0 0 0"/>
+        <xacro:inertial_box mass="${chassis_mass}" x="${chassis_length}" y="${chassis_width}" z="${chassis_height}">
+            <origin xyz="0 0 0" rpy="0 0 0"/>
         </xacro:inertial_box>
     </link>
     <gazebo reference="chassis">
-        <material>Gazebo/Orange</material>
+        <material>Gazebo/White</material>
     </gazebo>
     <!-- FRONT-LEFT WHEEL LINK -->
@@ -69,5 +60,5 @@
         <parent link="base_link"/>
         <child link="front_left_wheel"/>
-        <origin xyz="${wheel_offset_x} ${wheel_offset_y} ${wheel_offset_z}" rpy="-${pi/2} 0 0" />
+        <origin xyz="${wheel_offset_x} ${wheel_offset_y} ${-chassis_height/2}" rpy="-${pi/2} 0 0" />
         <axis xyz="0 0 1"/>
     </joint>
@@ -95,5 +86,5 @@
         <parent link="base_link"/>
         <child link="front_right_wheel"/>
-        <origin xyz="${wheel_offset_x} ${-wheel_offset_y} ${wheel_offset_z}" rpy="${pi/2} 0 0" />
+        <origin xyz="${wheel_offset_x} ${-wheel_offset_y} ${-chassis_height/2}" rpy="${pi/2} 0 0" />
         <axis xyz="0 0 -1"/>
     </joint>
@@ -121,5 +112,5 @@
         <parent link="base_link"/>
         <child link="rear_left_wheel"/>
-        <origin xyz="${-wheel_offset_x} ${wheel_offset_y} ${wheel_offset_z}" rpy="-${pi/2} 0 0" />
+        <origin xyz="${-wheel_offset_x} ${wheel_offset_y} ${-chassis_height/2}" rpy="-${pi/2} 0 0" />
         <axis xyz="0 0 1"/>
     </joint>
@@ -147,5 +138,5 @@
         <parent link="base_link"/>
         <child link="rear_right_wheel"/>
-        <origin xyz="${-wheel_offset_x} ${-wheel_offset_y} ${wheel_offset_z}" rpy="${pi/2} 0 0" />
+        <origin xyz="${-wheel_offset_x} ${-wheel_offset_y} ${-chassis_height/2}" rpy="${pi/2} 0 0" />
         <axis xyz="0 0 -1"/>
     </joint>
