Commit message: Added lidar sensor and scanned the world

File: description/lidar.xacro (robot description, xacro)
@@ -1,20 +1,19 @@
 <?xml version="1.0"?>
 <robot xmlns:xacro="http://www.ros.org/wiki/xacro" >
+    <xacro:property name="lidar_radius" value="0.03"/>
+    <xacro:property name="lidar_height" value="0.025"/>
+    <xacro:property name="lidar_mass" value="0.17"/>
+    <xacro:property name="lidar_offset_z" value="0.0625"/>
+    <xacro:property name="lidar_min_range" value="0.3"/>
+    <xacro:property name="lidar_max_range" value="12.0"/>
     <joint name="laser_joint" type="fixed">
         <parent link="chassis"/>
         <child link="laser_frame"/>
-        <origin xyz="0 0 0.10" rpy="0 0 0"/>
+        <origin xyz="0 0 ${lidar_offset_z}" rpy="0 0 0"/>
     </joint>
     <link name="laser_frame">
         <visual>
             <geometry>
-                <cylinder radius="0.05" length="0.04"/>
-            </geometry>
-            <material name="black"/>
-        </visual>
-        <visual>
-            <origin xyz="0 0 -0.03"/>
-            <geometry>
-                <cylinder radius="0.01" length="0.02"/>
+                <cylinder radius="${lidar_radius}" length="${lidar_height}"/>
             </geometry>
             <material name="black"/>
@@ -22,8 +21,8 @@
         <collision>
             <geometry>
-                <cylinder radius="0.05" length="0.04"/>
+                <cylinder radius="${lidar_radius}" length="${lidar_height}"/>
             </geometry>
         </collision>
-        <xacro:inertial_cylinder mass="0.1" length="0.04" radius="0.05">
+        <xacro:inertial_cylinder mass="${lidar_mass}" length="${lidar_height}" radius="${lidar_radius}">
             <origin xyz="0 0 0" rpy="0 0 0"/>
         </xacro:inertial_cylinder>
@@ -31,7 +30,8 @@
     <gazebo reference="laser_frame">
         <material>Gazebo/Black</material>
-        <sensor name="laser" type="ray">
+        <sensor name="rplidar" type="ray">
             <pose> 0 0 0 0 0 0 </pose>
-            <visualize>false</visualize>
+            <visualize>true</visualize>
+            <always_on>true</always_on>
             <update_rate>10</update_rate>
             <ray>
@@ -44,11 +44,11 @@
                 </scan>
                 <range>
-                    <min>0.3</min>
-                    <max>12</max>
+                    <min>${lidar_min_range}</min>
+                    <max>${lidar_max_range}</max>
                 </range>
             </ray>
             <plugin name="laser_controller" filename="libgazebo_ros_ray_sensor.so">
                 <ros>
-                    <argument>~/out:=scan</argument>
+                    <argument>--ros-args --remap ~/out:=scan</argument>
                 </ros>
                 <output_type>sensor_msgs/LaserScan</output_type>

Commit message: Added ros2_control and updated relevant files

File: description/lidar.xacro (robot description, xacro)
@@ -3,5 +3,5 @@
     <xacro:property name="lidar_radius" value="0.03"/>
     <xacro:property name="lidar_height" value="0.025"/>
-    <xacro:property name="lidar_mass" value="0.17"/>
+    <xacro:property name="lidar_mass" value="0.200"/>
     <xacro:property name="lidar_offset_z" value="0.0625"/>
     <xacro:property name="lidar_min_range" value="0.3"/>

File: description/robot.urdf.xacro (robot description, xacro)
@@ -1,6 +1,13 @@
 <?xml version="1.0"?>
 <robot xmlns:xacro="http://www.ros.org/wiki/xacro"  name="robot">
+    <xacro:arg name="use_ros2_control" default="true"/>
+    <xacro:arg name="sim_mode" default="true"/>
     <xacro:include filename="robot_core.xacro" />
-    <xacro:include filename="gazebo_control.xacro" />
+    <xacro:if value="$(arg use_ros2_control)">
+        <xacro:include filename="ros2_control.xacro" />
+    </xacro:if>
+    <xacro:unless value="$(arg use_ros2_control)">
+        <xacro:include filename="gazebo_control.xacro" />
+    </xacro:unless>
     <xacro:include filename="lidar.xacro" />
 </robot>

File: description/robot_core.xacro (robot description, xacro)
@@ -9,5 +9,5 @@
     <xacro:property name="wheel_thickness" value="0.020"/>
     <xacro:property name="wheel_mass" value="0.050"/>
-    <xacro:property name="wheel_offset_x" value="0.075"/>
+    <xacro:property name="wheel_offset_x" value="0.050"/>
     <xacro:property name="wheel_offset_y" value="0.070"/>
     <material name="white">

File: description/ros2_control.xacro (robot description, xacro)
@@ -36,5 +36,5 @@
                 <plugin>gazebo_ros2_control/GazeboSystem</plugin>
             </hardware>
-            <joint name="left_wheel_joint">
+            <joint name="front_left_wheel_joint">
                 <command_interface name="velocity">
                     <param name="min">-10</param>
@@ -44,5 +44,21 @@
                 <state_interface name="position"/>
             </joint>
-            <joint name="right_wheel_joint">
+            <joint name="front_right_wheel_joint">
+                <command_interface name="velocity">
+                    <param name="min">-10</param>
+                    <param name="max">10</param>
+                </command_interface>
+                <state_interface name="velocity"/>
+                <state_interface name="position"/>
+            </joint>
+            <joint name="rear_left_wheel_joint">
+                <command_interface name="velocity">
+                    <param name="min">-10</param>
+                    <param name="max">10</param>
+                </command_interface>
+                <state_interface name="velocity"/>
+                <state_interface name="position"/>
+            </joint>
+            <joint name="rear_right_wheel_joint">
                 <command_interface name="velocity">
                     <param name="min">-10</param>
@@ -57,5 +73,4 @@
         <plugin name="gazebo_ros2_control" filename="libgazebo_ros2_control.so">
             <parameters>$(find libot)/config/my_controllers.yaml</parameters>
-            <parameters>$(find libot)/config/gaz_ros2_ctl_use_sim.yaml</parameters>
         </plugin>
     </gazebo>

Commit message: Removed unnecessary files and optimized some code snippets for conciseness

File: description/lidar.xacro (robot description, xacro)
@@ -50,5 +50,5 @@
             <plugin name="laser_controller" filename="libgazebo_ros_ray_sensor.so">
                 <ros>
-                    <argument>--ros-args --remap ~/out:=scan</argument>
+                    <argument>~/out:=scan</argument>
                 </ros>
                 <output_type>sensor_msgs/LaserScan</output_type>

File: description/robot_core.xacro (robot description, xacro)
@@ -14,20 +14,31 @@
         <color rgba="1 1 1 1" />
     </material>
-    <material name="orange">
-        <color rgba="1 0.3 0.1 1"/>
+    <material name="grey">
+        <color rgba="0.4 0.4 0.4 1"/>
+    </material>
+    <material name="black">
+        <color rgba="0 0 0 1"/>
     </material>
     <material name="blue">
         <color rgba="0.2 0.2 1 1"/>
     </material>
-    <material name="black">
-        <color rgba="0 0 0 1"/>
-    </material>
     <material name="red">
         <color rgba="1 0 0 1"/>
+    </material>
+    <material name="yellow">
+        <color rgba="1 1 0 1"/>
     </material>
     <!-- BASE LINK -->
     <link name="base_link">
     </link>
-    <!-- CHASSIS LINK -->
+    <!-- BASE_FOOTPRINT LINK -->
+    <joint name="base_footprint_joint" type="fixed">
+        <parent link="base_link"/>
+        <child link="base_footprint"/>
+        <origin xyz="0 0 0" rpy="0 0 0"/>
+    </joint>
+    <link name="base_footprint">
+    </link>
+    <!-- CHASSIS -->
     <joint name="chassis_joint" type="fixed">
         <parent link="base_link"/>
@@ -41,5 +52,5 @@
                 <box size="${chassis_length} ${chassis_width} ${chassis_height}"/>
             </geometry>
-            <material name="white"/>
+            <material name="grey"/>
         </visual>
         <collision>
@@ -54,109 +65,41 @@
     </link>
     <gazebo reference="chassis">
-        <material>Gazebo/White</material>
+        <material>Gazebo/Grey</material>
     </gazebo>
-    <!-- FRONT-LEFT WHEEL LINK -->
-    <joint name="front_left_wheel_joint" type="continuous">
-        <parent link="base_link"/>
-        <child link="front_left_wheel"/>
-        <origin xyz="${wheel_offset_x} ${wheel_offset_y} ${-chassis_height/2}" rpy="-${pi/2} 0 0" />
-        <axis xyz="0 0 1"/>
-    </joint>
-    <link name="front_left_wheel">
-        <visual>
-            <geometry>
-                <cylinder radius="${wheel_radius}" length="${wheel_thickness}"/>
-            </geometry>
-            <material name="blue"/>
-        </visual>
-        <collision>
-            <geometry>
-                <sphere radius="${wheel_radius}"/>
-            </geometry>
-        </collision>
-        <xacro:inertial_cylinder mass="${wheel_mass}" length="${wheel_thickness}" radius="${wheel_radius}">
-            <origin xyz="0 0 0" rpy="0 0 0"/>
-        </xacro:inertial_cylinder>
-    </link>
-    <gazebo reference="front_left_wheel">
-        <material>Gazebo/Blue</material>
-    </gazebo>
-    <!-- FRONT-RIGHT WHEEL LINK -->
-    <joint name="front_right_wheel_joint" type="continuous">
-        <parent link="base_link"/>
-        <child link="front_right_wheel"/>
-        <origin xyz="${wheel_offset_x} ${-wheel_offset_y} ${-chassis_height/2}" rpy="${pi/2} 0 0" />
-        <axis xyz="0 0 -1"/>
-    </joint>
-    <link name="front_right_wheel">
-        <visual>
-            <geometry>
-                <cylinder radius="${wheel_radius}" length="${wheel_thickness}"/>
-            </geometry>
-            <material name="blue"/>
-        </visual>
-        <collision>
-            <geometry>
-                <sphere radius="${wheel_radius}"/>
-            </geometry>
-        </collision>
-        <xacro:inertial_cylinder mass="${wheel_mass}" length="${wheel_thickness}" radius="${wheel_radius}">
-            <origin xyz="0 0 0" rpy="0 0 0"/>
-        </xacro:inertial_cylinder>
-    </link>
-    <gazebo reference="front_right_wheel">
-        <material>Gazebo/Blue</material>
-    </gazebo>
-    <!-- REAR-LEFT WHEEL LINK -->
-    <joint name="rear_left_wheel_joint" type="continuous">
-        <parent link="base_link"/>
-        <child link="rear_left_wheel"/>
-        <origin xyz="${-wheel_offset_x} ${wheel_offset_y} ${-chassis_height/2}" rpy="-${pi/2} 0 0" />
-        <axis xyz="0 0 1"/>
-    </joint>
-    <link name="rear_left_wheel">
-        <visual>
-            <geometry>
-                <cylinder radius="${wheel_radius}" length="${wheel_thickness}"/>
-            </geometry>
-            <material name="blue"/>
-        </visual>
-        <collision>
-            <geometry>
-                <sphere radius="${wheel_radius}"/>
-            </geometry>
-        </collision>
-        <xacro:inertial_cylinder mass="${wheel_mass}" length="${wheel_thickness}" radius="${wheel_radius}">
-            <origin xyz="0 0 0" rpy="0 0 0"/>
-        </xacro:inertial_cylinder>
-    </link>
-    <gazebo reference="rear_left_wheel">
-        <material>Gazebo/Blue</material>
-    </gazebo>
-    <!-- REAR-RIGHT WHEEL LINK -->
-    <joint name="rear_right_wheel_joint" type="continuous">
-        <parent link="base_link"/>
-        <child link="rear_right_wheel"/>
-        <origin xyz="${-wheel_offset_x} ${-wheel_offset_y} ${-chassis_height/2}" rpy="${pi/2} 0 0" />
-        <axis xyz="0 0 -1"/>
-    </joint>
-    <link name="rear_right_wheel">
-        <visual>
-            <geometry>
-                <cylinder radius="${wheel_radius}" length="${wheel_thickness}"/>
-            </geometry>
-            <material name="blue"/>
-        </visual>
-        <collision>
-            <geometry>
-                <sphere radius="${wheel_radius}"/>
-            </geometry>
-        </collision>
-        <xacro:inertial_cylinder mass="${wheel_mass}" length="${wheel_thickness}" radius="${wheel_radius}">
-            <origin xyz="0 0 0" rpy="0 0 0"/>
-        </xacro:inertial_cylinder>
-    </link>
-    <gazebo reference="rear_right_wheel">
-        <material>Gazebo/Blue</material>
-    </gazebo>
+    <!-- WHEELS -->
+    <xacro:macro name="wheel" params="name x y axis rpy_axis">
+        <joint name="${name}_joint" type="continuous">
+            <parent link="base_link"/>
+            <child link="${name}"/>
+            <origin xyz="${x} ${y} ${-chassis_height/2}" rpy="${rpy_axis}" />
+            <axis xyz="${axis}"/>
+        </joint>
+        <link name="${name}">
+            <visual>
+                <geometry>
+                    <cylinder radius="${wheel_radius}" length="${wheel_thickness}"/>
+                </geometry>
+                <material name="yellow"/>
+            </visual>
+            <collision>
+                <geometry>
+                    <sphere radius="${wheel_radius}"/>
+                </geometry>
+            </collision>
+            <xacro:inertial_cylinder mass="${wheel_mass}" length="${wheel_thickness}" radius="${wheel_radius}">
+                <origin xyz="0 0 0" rpy="0 0 0"/>
+            </xacro:inertial_cylinder>
+        </link>
+        <gazebo reference="${name}">
+            <material>Gazebo/Yellow</material>
+        </gazebo>
+    </xacro:macro>
+    <!-- Front Left Wheel -->
+    <xacro:wheel name="front_left_wheel" x="${wheel_offset_x}" y="${wheel_offset_y}" axis="0 0 1" rpy_axis="-${pi/2} 0 0"/>
+    <!-- Front Right Wheel -->
+    <xacro:wheel name="front_right_wheel" x="${wheel_offset_x}" y="-${wheel_offset_y}" axis="0 0 -1" rpy_axis="${pi/2} 0 0"/>
+    <!-- Rear Left Wheel -->
+    <xacro:wheel name="rear_left_wheel" x="-${wheel_offset_x}" y="${wheel_offset_y}" axis="0 0 1" rpy_axis="-${pi/2} 0 0"/>
+    <!-- Rear Right Wheel -->
+    <xacro:wheel name="rear_right_wheel" x="-${wheel_offset_x}" y="-${wheel_offset_y}" axis="0 0 -1" rpy_axis="${pi/2} 0 0"/>
 </robot>

File: description/ros2_control.xacro (robot description, xacro)
@@ -1,4 +1,16 @@
 <?xml version="1.0"?>
 <robot xmlns:xacro="http://www.ros.org/wiki/xacro">
+    <!-- Define the joint configuration of the wheels for both real robot and simulated one -->
+    <xacro:macro name="wheel_joint_config" params="joint_name">
+        <joint name="${joint_name}">
+            <command_interface name="velocity">
+                <param name="min">-10</param>
+                <param name="max">10</param>
+            </command_interface>
+            <state_interface name="velocity"/>
+            <state_interface name="position"/>
+        </joint>
+    </xacro:macro>
+    <!-- Real Robot Control -->
     <xacro:unless value="$(arg sim_mode)">
         <ros2_control name="RealRobot" type="system">
@@ -13,22 +25,10 @@
                 <param name="enc_counts_per_rev">3436</param>
             </hardware>
-            <joint name="left_wheel_joint">
-                <command_interface name="velocity">
-                    <param name="min">-10</param>
-                    <param name="max">10</param>
-                </command_interface>
-                <state_interface name="velocity"/>
-                <state_interface name="position"/>
-            </joint>
-            <joint name="right_wheel_joint">
-                <command_interface name="velocity">
-                    <param name="min">-10</param>
-                    <param name="max">10</param>
-                </command_interface>
-                <state_interface name="velocity"/>
-                <state_interface name="position"/>
-            </joint>
+            <xacro:foreach items="front_left_wheel_joint front_right_wheel_joint rear_left_wheel_joint rear_right_wheel_joint" as="joint">
+                <xacro:wheel_joint_config joint_name="${joint}"/>
+            </xacro:foreach>
         </ros2_control>
     </xacro:unless>
+    <!-- Simulated Robot Control -->
     <xacro:if value="$(arg sim_mode)">
         <ros2_control name="GazeboSystem" type="system">
@@ -36,38 +36,10 @@
                 <plugin>gazebo_ros2_control/GazeboSystem</plugin>
             </hardware>
-            <joint name="front_left_wheel_joint">
-                <command_interface name="velocity">
-                    <param name="min">-10</param>
-                    <param name="max">10</param>
-                </command_interface>
-                <state_interface name="velocity"/>
-                <state_interface name="position"/>
-            </joint>
-            <joint name="front_right_wheel_joint">
-                <command_interface name="velocity">
-                    <param name="min">-10</param>
-                    <param name="max">10</param>
-                </command_interface>
-                <state_interface name="velocity"/>
-                <state_interface name="position"/>
-            </joint>
-            <joint name="rear_left_wheel_joint">
-                <command_interface name="velocity">
-                    <param name="min">-10</param>
-                    <param name="max">10</param>
-                </command_interface>
-                <state_interface name="velocity"/>
-                <state_interface name="position"/>
-            </joint>
-            <joint name="rear_right_wheel_joint">
-                <command_interface name="velocity">
-                    <param name="min">-10</param>
-                    <param name="max">10</param>
-                </command_interface>
-                <state_interface name="velocity"/>
-                <state_interface name="position"/>
-            </joint>
+            <xacro:foreach items="front_left_wheel_joint front_right_wheel_joint rear_left_wheel_joint rear_right_wheel_joint" as="joint">
+                <xacro:wheel_joint_config joint_name="${joint}"/>
+            </xacro:foreach>
         </ros2_control>
     </xacro:if>
+    <!-- Gazebo Plugin -->
     <gazebo>
         <plugin name="gazebo_ros2_control" filename="libgazebo_ros2_control.so">

Commit message: Adjusted some parameters to match the real

File: description/lidar.xacro (robot description, xacro)
@@ -1,8 +1,8 @@
 <?xml version="1.0"?>
 <robot xmlns:xacro="http://www.ros.org/wiki/xacro" >
-    <xacro:property name="lidar_radius" value="0.03"/>
-    <xacro:property name="lidar_height" value="0.025"/>
-    <xacro:property name="lidar_mass" value="0.200"/>
-    <xacro:property name="lidar_offset_z" value="0.0625"/>
+    <xacro:property name="lidar_radius" value="0.035"/>
+    <xacro:property name="lidar_height" value="0.030"/>
+    <xacro:property name="lidar_mass" value="0.175"/>
+    <xacro:property name="lidar_offset_z" value="0.085"/>
     <xacro:property name="lidar_min_range" value="0.3"/>
     <xacro:property name="lidar_max_range" value="12.0"/>

File: description/robot_core.xacro (robot description, xacro)
@@ -2,13 +2,13 @@
 <robot xmlns:xacro="http://www.ros.org/wiki/xacro" >
     <xacro:include filename="inertial_macros.xacro"/>
-    <xacro:property name="chassis_length" value="0.24"/>
-    <xacro:property name="chassis_width" value="0.12"/>
-    <xacro:property name="chassis_height" value="0.10"/>
-    <xacro:property name="chassis_mass" value="0.800"/>
-    <xacro:property name="wheel_radius" value="0.025"/>
-    <xacro:property name="wheel_thickness" value="0.020"/>
+    <xacro:property name="chassis_length" value="0.230"/>
+    <xacro:property name="chassis_width" value="0.105"/>
+    <xacro:property name="chassis_height" value="0.090"/>
+    <xacro:property name="chassis_mass" value="0.725"/>
+    <xacro:property name="wheel_radius" value="0.0325"/>
+    <xacro:property name="wheel_thickness" value="0.025"/>
     <xacro:property name="wheel_mass" value="0.050"/>
-    <xacro:property name="wheel_offset_x" value="0.050"/>
-    <xacro:property name="wheel_offset_y" value="0.070"/>
+    <xacro:property name="wheel_offset_x" value="0.040"/>
+    <xacro:property name="wheel_offset_y" value="0.065"/>
     <material name="white">
         <color rgba="1 1 1 1" />
@@ -72,5 +72,5 @@
             <parent link="base_link"/>
             <child link="${name}"/>
-            <origin xyz="${x} ${y} ${-chassis_height/2}" rpy="${rpy_axis}" />
+            <origin xyz="${x} ${y} ${-chassis_height/2 + 0.015}" rpy="${rpy_axis}" />
             <axis xyz="${axis}"/>
         </joint>

Commit message: new changes post 3 battery supply

File: description/lidar.xacro (robot description, xacro)
@@ -10,5 +10,5 @@
         <parent link="chassis"/>
         <child link="laser_frame"/>
-        <origin xyz="0 0 ${lidar_offset_z}" rpy="0 0 0"/>
+        <origin xyz="0 0 ${lidar_offset_z}" rpy="0 0 ${pi}"/>
     </joint>
     <link name="laser_frame">

File: description/robot_core.xacro (robot description, xacro)
@@ -5,5 +5,5 @@
     <xacro:property name="chassis_width" value="0.105"/>
     <xacro:property name="chassis_height" value="0.090"/>
-    <xacro:property name="chassis_mass" value="0.725"/>
+    <xacro:property name="chassis_mass" value="0.825"/>
     <xacro:property name="wheel_radius" value="0.0325"/>
     <xacro:property name="wheel_thickness" value="0.025"/>
